File: hardware/board/solder-reflow/solder-reflow.kicad_sch (KiCad schematic)
At the start: 38 parts, among them J1 AC_Con, J2 OLED 0.91, Q1 BC557, SW1 RotaryEncoder_Switch, U1 OPA2134, U2 WeMos_D1_mini, U3 S202S02, U4 OPA2134, U5 TL431D

Commit message: finish pcb layout
add a backup zip
Parts:
- removed U3: S202S02, Package_SIP:SIP4_Sharp-SSR_P7.62mm_Straight, symbol Relay_SolidState:S202S02
- removed U5: TL431D, Package_SO:SOIC-8_3.9x4.9mm_P1.27mm, symbol Reference_Voltage:TL431D
- added C6: 0.33uF, Capacitor_THT:CP_Radial_D6.3mm_P2.50mm, symbol Device:C_Polarized
- added C7: 0.1uF, Capacitor_THT:CP_Radial_D6.3mm_P2.50mm, symbol Device:C_Polarized
- added D2: SSR, LED_THT:LED_D5.0mm, symbol Device:LED
- added D3: POWER_LED, LED_THT:LED_D5.0mm, symbol Device:LED
- added H1, H2, H3, H4, H5: MountingHole_Pad, MountingHole:MountingHole_3.2mm_M3_DIN965_Pad, symbol Mechanical:MountingHole_Pad
- added J3: PTC_Con, TerminalBlock_MetzConnect:TerminalBlock_MetzConnect_Type011_RT05502HBWC_1x02_P5.00mm_Horizontal, symbol Connector:Screw_Terminal_01x02
- added J4: Barrel_Jack_Switch_Pin3Ring, Connector_BarrelJack:BarrelJack_Horizontal, symbol Connector:Barrel_Jack_Switch_Pin3Ring
- added K1: G3MB202PDC12, downloadedLibrary:RELAY_G3MB202PDC12, symbol G3MB202PDC12:G3MB202PDC12
- added R22: 1k, Resistor_THT:R_Axial_DIN0207_L6.3mm_D2.5mm_P10.16mm_Horizontal, symbol Device:R_US
- added U1: TL431LP, Package_TO_SOT_THT:TO-92_Inline_Wide, symbol Reference_Voltage:TL431LP
- added U4: L7805, Package_TO_SOT_THT:TO-220F-3_Horizontal_TabDown, symbol Regulator_Linear:L7805
- C1: renamed from C3; footprint (none) -> Capacitor_THT:C_Disc_D4.3mm_W1.9mm_P5.00mm
- C2, C4, C5: footprint (none) -> Capacitor_THT:C_Disc_D4.3mm_W1.9mm_P5.00mm
- C3: renamed from C1; footprint (none) -> Capacitor_THT:C_Disc_D4.3mm_W1.9mm_P5.00mm
- F1: footprint (none) -> Fuse:Fuseholder_Littelfuse_100_series_5x30mm
- Q1: footprint Package_TO_SOT_THT:TO-92_Inline -> Package_TO_SOT_THT:TO-92_Inline_Wide
- R1: renamed from R11; footprint (none) -> Resistor_THT:R_Axial_DIN0207_L6.3mm_D2.5mm_P10.16mm_Horizontal
- R10: renamed from R20; footprint (none) -> Resistor_THT:R_Axial_DIN0207_L6.3mm_D2.5mm_P10.16mm_Horizontal
- R11: renamed from R21; footprint (none) -> Resistor_THT:R_Axial_DIN0207_L6.3mm_D2.5mm_P10.16mm_Horizontal
- R12: renamed from R7; footprint (none) -> Resistor_THT:R_Axial_DIN0207_L6.3mm_D2.5mm_P10.16mm_Horizontal
- R13: renamed from R6; footprint (none) -> Resistor_THT:R_Axial_DIN0207_L6.3mm_D2.5mm_P10.16mm_Horizontal
- R14: renamed from R13; footprint (none) -> Resistor_THT:R_Axial_DIN0207_L6.3mm_D2.5mm_P10.16mm_Horizontal
- R15: renamed from R12; footprint (none) -> Resistor_THT:R_Axial_DIN0207_L6.3mm_D2.5mm_P10.16mm_Horizontal
- R16, R19: footprint (none) -> Resistor_THT:R_Axial_DIN0207_L6.3mm_D2.5mm_P10.16mm_Horizontal
- R17: renamed from R15; footprint (none) -> Resistor_THT:R_Axial_DIN0207_L6.3mm_D2.5mm_P10.16mm_Horizontal
- R18: renamed from R14; footprint (none) -> Resistor_THT:R_Axial_DIN0207_L6.3mm_D2.5mm_P10.16mm_Horizontal
- R2: renamed from R1; footprint (none) -> Resistor_THT:R_Axial_DIN0207_L6.3mm_D2.5mm_P10.16mm_Horizontal
- R20: renamed from R17; footprint (none) -> Resistor_THT:R_Axial_DIN0207_L6.3mm_D2.5mm_P10.16mm_Horizontal
- R21: renamed from R18; footprint (none) -> Resistor_THT:R_Axial_DIN0207_L6.3mm_D2.5mm_P10.16mm_Horizontal
- R3: renamed from R5; footprint (none) -> Resistor_THT:R_Axial_DIN0207_L6.3mm_D2.5mm_P10.16mm_Horizontal
- R4: renamed from R2; footprint (none) -> Resistor_THT:R_Axial_DIN0207_L6.3mm_D2.5mm_P10.16mm_Horizontal
- R5: renamed from R4; footprint (none) -> Resistor_THT:R_Axial_DIN0207_L6.3mm_D2.5mm_P10.16mm_Horizontal
- R6: renamed from R3; footprint (none) -> Resistor_THT:R_Axial_DIN0207_L6.3mm_D2.5mm_P10.16mm_Horizontal
- R7: renamed from R8; footprint (none) -> Resistor_THT:R_Axial_DIN0207_L6.3mm_D2.5mm_P10.16mm_Horizontal
- R8: renamed from R9; footprint (none) -> Resistor_THT:R_Axial_DIN0207_L6.3mm_D2.5mm_P10.16mm_Horizontal
- R9: renamed from R10; footprint (none) -> Resistor_THT:R_Axial_DIN0207_L6.3mm_D2.5mm_P10.16mm_Horizontal
- SW1: footprint (none) -> Rotary_Encoder:RotaryEncoder_Alps_EC11E-Switch_Vertical_H20mm
- renumbered U1 to U2, U4 to U3, U2 to U5
Connections:
- net +2V5: now also U1.1 (REF), U1.3 (K)
- net +5V: now also C7.1, R22.2, U4.3 (OUT)
- net GND: now also C6.2, C7.2, D2.1 (K), D3.1 (K), J3.2 (Pin_2), J4.2, J4.3, K1.4 (-), U1.2 (A), U4.2 (GND); no longer R18.1
- net pt100_out: now also J3.1 (Pin_1)
- net at Q1.1 (C), R18.2: now also K1.3 (+)
- net at F1.1: now also K1.2 (L2)
- net at J1.2 (Pin_2): now also K1.1 (L1)
- new net: D2.2 (A), R18.1
- new net: C6.1, J4.1, U4.1 (IN)
- new net: D3.2 (A), R22.1
- no-connect marks 0 -> 5
Other:
- note added: "PT100/RTD Signal Conditioning"
- note added: "Voltage Regulator"
- note removed: "PT100 Signal Conditioning"
- moved on the sheet: C4, C5, D1, F1, J1, Q1, R14, R15, R16, R17, R18, R19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
