File: hardware/board/solder-reflow.kicad_sch (KiCad schematic)
At the start: 51 parts, among them J1 AC_Con, J2 OLED 0.91, J3 PTC_Con, J4 Barrel_Jack_Switch_Pin3Ring, K1 G3MB202PDC12, Q1 BC557, SW1 RotaryEncoder_Switch, U1 TL431LP, U2 OPA2134, U3 OPA2134, U4 L7805, U5 WeMos_D1_mini

Commit message: [5-6-0014] adding several io connection
Parts:
- removed Q1: BC557, Package_TO_SOT_THT:TO-92_Inline_Wide, symbol Transistor_BJT:BC557
- removed U2, U3: OPA2134, Package_DIP:DIP-8_W7.62mm_LongPads, symbol Amplifier_Operational:OPA2134
- added C10, C11, C12, C14, C15: 100nF, Capacitor_THT:C_Disc_D4.3mm_W1.9mm_P5.00mm, symbol Device:C
- added C13, C8, C9: 22uF, Capacitor_THT:C_Disc_D4.3mm_W1.9mm_P5.00mm, symbol Device:C
- added C16, C17, C18, C19: 1uF, Capacitor_THT:C_Disc_D4.3mm_W1.9mm_P5.00mm, symbol Device:C
- added D4: 1N4001, Diode_THT:D_DO-41_SOD81_P10.16mm_Horizontal, symbol Diode:1N4001
- added D5: SSR2, LED_THT:LED_D5.0mm, symbol Device:LED
- added D6: 3.3VPWR, LED_THT:LED_D5.0mm, symbol Device:LED
- added D7: TXD, LED_THT:LED_D5.0mm, symbol Device:LED
- added D8: RXD, LED_THT:LED_D5.0mm, symbol Device:LED
- added J10, J7, J8, J9: PINOUT1, Connector_PinSocket_2.54mm:PinSocket_1x08_P2.54mm_Vertical, symbol Connector_Generic:Conn_01x08
- added J5: SSROUT2, TerminalBlock_MetzConnect:TerminalBlock_MetzConnect_Type011_RT05502HBWC_1x02_P5.00mm_Horizontal, symbol Connector:Screw_Terminal_01x02
- added J6: USB_B, symbol Connector:USB_B
- added Q1, Q2: SS8550, Package_TO_SOT_SMD:SOT-23_Handsoldering, symbol Transistor_BJT:BC807
- added Q3, Q4: SS8050, Package_TO_SOT_SMD:SOT-23_Handsoldering, symbol Transistor_BJT:BC817
- added R23, R24: 10k, Resistor_SMD:R_0805_2012Metric_Pad1.20x1.40mm_HandSolder, symbol Device:R_US
- added R25, R26, R27, R28: 1k, Resistor_SMD:R_0805_2012Metric_Pad1.20x1.40mm_HandSolder, symbol Device:R_US
- added R29, R30, R31, R32: 22k, Resistor_SMD:R_0805_2012Metric_Pad1.20x1.40mm_HandSolder, symbol Device:R_US
- added SW2: RST, symbol Switch:SW_Push
- added SW3, SW4, SW5, SW6, SW7: IO0, symbol Switch:SW_Push
- added U2: TL074, Package_SO:SOIC-14_3.9x8.7mm_P1.27mm, symbol Amplifier_Operational:TL074
- added U3: AMS1117-3.3, Package_TO_SOT_SMD:SOT-223-3_TabPin2, symbol Regulator_Linear:AMS1117-3.3
- added U6: ESP32-WROOM-32D, RF_Module:ESP32-WROOM-32D, symbol RF_Module:ESP32-WROOM-32D
- added U7: CH340C, Package_SO:SOIC-16_3.9x9.9mm_P1.27mm, symbol Interface_USB:CH340C
- D2: value SSR -> SSR1
- J1: value AC_Con -> AC_Con1
- R1, R12, R13, R14, R15, R16, R17, R18, R19, R2, R20, R21, R22, R3, R4, R5, R6, R8, R9: footprint Resistor_THT:R_Axial_DIN0207_L6.3mm_D2.5mm_P10.16mm_Horizontal -> Resistor_SMD:R_0805_2012Metric_Pad1.20x1.40mm_HandSolder
- R10: value 5.1K -> 10k; footprint Resistor_THT:R_Axial_DIN0207_L6.3mm_D2.5mm_P10.16mm_Horizontal -> Resistor_SMD:R_0805_2012Metric_Pad1.20x1.40mm_HandSolder
- R11: value 10k -> 1k; footprint Resistor_THT:R_Axial_DIN0207_L6.3mm_D2.5mm_P10.16mm_Horizontal -> Resistor_SMD:R_0805_2012Metric_Pad1.20x1.40mm_HandSolder
- R7: value 1k -> 10k; footprint Resistor_THT:R_Axial_DIN0207_L6.3mm_D2.5mm_P10.16mm_Horizontal -> Resistor_SMD:R_0805_2012Metric_Pad1.20x1.40mm_HandSolder
Connections:
- net +2V5: now also R1.1; no longer R1.2
- net +5V: now also R1.2, C8.1, D4.2 (A), J6.1 (VBUS), U2.4 (V+), U3.3 (VI); no longer R1.1
- net GND: now also C10.2, C11.2, C12.2, C13.2, C14.2, C15.2, C16.2, C17.2, C18.2, C19.2, C8.2, C9.2, D5.1 (K), D6.1 (K), J5.2 (Pin_2), J6.4 (GND), J6.5 (Shield), SW2.1, SW3.1, SW4.1, SW5.1, SW6.1, SW7.1, U2.11 (V-), U3.1 (GND), U6.1 (GND), U6.15 (GND), U6.38 (GND), U6.39 (GND), U7.1 (GND); no longer R11.1
- net SSR_in: no longer R15.1
- net at R12.2, R13.1: now also U2.9 (-)
- net at C3.1, R9.1: now also U2.10 (+)
- net at K1.3 (+), R18.2: now also Q1.3 (C)
- net at R4.2: now also U2.6 (-), U2.7
- net at R5.2, R6.2: now also U2.2 (-)
- net at R11.2: now also D6.2 (A); no longer R10.2
- net at R3.2, R6.1: now also U2.1
- net at R2.2, R4.1: now also U2.3 (+)
- net at R14.1, R15.2: now also Q1.1 (B)
- net at D1.1 (K), R14.2: now also Q1.2 (E)
- net at C1.1: now also R13.2, U2.12 (+), U2.8; no longer R7.2
- net pt100_out renamed PT100Voltage
- net PT100Voltage: now also U2.5 (+)
- new net: D4.1 (K), Q2.2 (E), R24.2
- new net: J6.3 (D+), U7.5 (UD+)
- new net: J6.2 (D-), U7.6 (UD-)
- new net: R32.2, SW7.2
- new net: D5.2 (A), R25.1
- new net: D7.2 (A), R26.2
- new net: R30.2, SW4.2
- new net: D8.2 (A), R27.2
- new net: Q3.1 (B), R7.1
- new net: R31.2, SW5.2
- new net: Q2.1 (B), R23.2, R24.1
- new net: J5.1 (Pin_1), Q2.3 (C), R25.2
- new net: Q4.1 (B), R10.1
- new net: R29.2, SW6.2
- new net +3.3V: C10.1, C12.1, C13.1, C9.1, R11.1, R26.1, R27.1, R28.1, U3.2 (VO), U6.2 (VDD), U7.16 (VCC), U7.4 (V3)
- new net ADC1_CH7: U6.7 (IO35)
- new net DTR: Q4.2 (E), R7.2, U7.13 (~{DTR})
- new net EN: C11.1, C14.1, Q3.3 (C), R28.2, SW2.2, U6.3 (EN)
- new net I2C_SCL: U6.28 (IO17)
- new net I2C_SDA: U6.27 (IO16)
- new net IN1: C18.1, R29.1, U6.12 (IO27)
- new net IN2: C16.1, R30.1, U6.11 (IO26)
- new net IN3: C17.1, R31.1, U6.10 (IO25)
- new net IN4: C19.1, R32.1, U6.36 (IO22)
- new net IO0: C15.1, Q4.3 (C), SW3.2, U6.25 (IO0)
- new net IO2: U6.24 (IO2)
- new net IO21: U6.33 (IO21)
- new net IO32: U6.8 (IO32)
- new net IO33: U6.9 (IO33)
- new net IO4: U6.26 (IO4)
- new net MTCK: U6.16 (IO13)
- new net MTDI: U6.14 (IO12)
- new net MTDO: U6.23 (IO15)
- new net MTMS: U6.13 (IO14)
- new net PT100: U2.13 (-), U2.14, U6.6 (IO34)
- new net RTS: Q3.2 (E), R10.2, U7.14 (~{RTS})
- new net RXD: D8.1 (K), U6.35 (TXD0/IO1), U7.3 (RXD)
- new net SSRIN1: R15.1
- new net SSRIN2: R23.1
- new net TXD: D7.1 (K), U6.34 (RXD0/IO3), U7.2 (TXD)
- new net VSPI_CLK: U6.30 (IO18)
- new net VSPI_CS0: U6.29 (IO5)
- new net VSPI_D: U6.37 (IO23)
- new net VSPI_Q: U6.31 (IO19)
- no-connect marks 11 -> 23
Other:
- note added: "JTAG Debugging, With OpenOCD https://docs.espressif.com/projects/esp-idf/en/latest/esp32/api-guides/jtag-debugging/index.html"
- note added: "Need To Add External Pull Up"
- note added: "Output is limited by output range, which is typically 1.5 V to 10.5 V, or VCC- + 1.5 V to VCC+ - 1.5 V."
- note added: "Pins SCK/CLK, SDO/SD0, SDI/SD1, SHD/SD2, SWP/SD3 and SCS/CMD, namely, GPIO6 to GPIO11 are connected to the integrated SPI flash integrated on the module and are not recommended for other uses."
- note added: "Reference Design Schematic: ESP32-DevKit V4 https://dl.espressif.com/dl/schematics/esp32_devkitc_v4-sch.pdf"
- note added: "SPI Terminology in ESP32 The spi_master driver uses the following terms: Host: The SPI peripheral inside the ESP32 initiating the SPI transmissions. One of SPI, HSPI or VSPI. (For now, only HSPI or VSPI are actually supported in the driver; it will support all 3 peripherals somewhere in the future.) Bus: The SPI bus, common to all SPI devices connected to one host. In general the bus consists of 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"
- note added: "Target Temp for PT100 is Less 400*C, Based on Resistance table its about 250ohm"
- note removed: "Voltage Divider 5 to 3.3"
- moved on the sheet: C1, D3, R1, R15, R22, R8, U1, U5

Commit message: [5-6-0703] adding st7789 schematic
Parts:
- removed C2: 390nF, Capacitor_THT:C_Disc_D4.3mm_W1.9mm_P5.00mm, symbol Device:C
- removed C4, C5: 10nF, Capacitor_THT:C_Disc_D4.3mm_W1.9mm_P5.00mm, symbol Device:C
- removed R16, R17, R19, R20, R21: 10k, Resistor_SMD:R_0805_2012Metric_Pad1.20x1.40mm_HandSolder, symbol Device:R_US
- removed SW1: RotaryEncoder_Switch, Rotary_Encoder:RotaryEncoder_Alps_EC11E-Switch_Vertical_H20mm, symbol Device:RotaryEncoder_Switch
- added J11: JTAG10, Connector_IDC:IDC-Header_2x10_P2.54mm_Vertical, symbol Connector:Conn_ARM_JTAG_SWD_10
- added J12: ST7789, Connector_PinSocket_2.54mm:PinSocket_1x07_P2.54mm_Vertical, symbol Connector_Generic:Conn_01x07
- added R12, R13: 4K7, Resistor_SMD:R_0805_2012Metric_Pad1.20x1.40mm_HandSolder, symbol Device:R_US
- C1: value 68nF -> 1nF
- C3: value 180nF -> 1nF
- R8: value 17.4k -> 16k
- R9: value 107k -> 16k
- RA: renamed from R13; value 20k -> 25k
- RB: renamed from R12; value 3.09k -> 25k
Connections:
- net IO21 is gone; now on net SSRIN2: U6.33 (IO21)
- net IO4 is gone; now on net SSRIN1: U6.26 (IO4)
- net +3.3V: now also J11.1 (VTref), J12.2 (Pin_2), J12.7 (Pin_7), R12.2, R13.2
- net EN: now also J11.10 (~{RESET})
- net GND: now also J11.3 (GND), J11.5 (GND), J11.9 (GNDDetect), J12.1 (Pin_1)
- net I2C_SCL: now also J2.2 (Pin_2), R13.1
- net I2C_SDA: now also J2.1 (Pin_1), R12.1
- net MTCK: now also J11.4 (SWCLK/TCK)
- net MTDI: now also J11.8 (NC/TDI)
- net MTDO: now also J11.6 (SWO/TDO)
- net MTMS: now also J11.2 (SWDIO/TMS)
- net OLED_SCL: no longer J2.1 (Pin_1)
- net OLED_SDA: no longer J2.2 (Pin_2)
- net VSPI_CLK: now also J12.3 (Pin_3)
- net VSPI_D: now also J12.4 (Pin_4)
- net IO32 renamed LCD_RST
- net LCD_RST: now also J12.5 (Pin_5)
- net IO33 renamed LCD_DC
- net LCD_DC: now also J12.6 (Pin_6)
Other:
- note added: "INPUT SWITCH"
- note added: "LCD_BACKLIGHT"
- note added: "Pinout Image https://electropeak.com/learn/wp-content/uploads/2021/02/1-3-Inch-240x240-IPS-SPI-HD-LCD-Full-Color-Display-OLED-Module-Pin.jpg"
- note added: "Sallen-Key Filter http://sim.okawa-denshi.jp/en/OPstool.php"
- note removed: "Rotary Encoder"
- note removed: "Sallen-Key Filter"
- moved on the sheet: C1, C11, C6, C7, J2, J4, R28, R8, U4

Commit message: [6-6-0359] finish first revision, need to review
Parts:
- removed J10, J7, J8, J9: PINOUT1, Connector_PinSocket_2.54mm:PinSocket_1x08_P2.54mm_Vertical, symbol Connector_Generic:Conn_01x08
- removed U5: WeMos_D1_mini, Module:WEMOS_D1_mini_light, symbol MCU_Module:WeMos_D1_mini
- added C2: 1uF, Capacitor_THT:C_Disc_D4.3mm_W1.9mm_P5.00mm, symbol Device:C
- added J10, J7, J8: PINOUT, Connector_PinHeader_2.54mm:PinHeader_1x10_P2.54mm_Vertical, symbol Connector_Generic:Conn_01x10
- added J9: 12VIN, TerminalBlock_MetzConnect:TerminalBlock_MetzConnect_Type011_RT05502HBWC_1x02_P5.00mm_Horizontal, symbol Connector:Screw_Terminal_01x02
- added R16, R17, R19, R20: 10k, Resistor_SMD:R_0805_2012Metric_Pad1.20x1.40mm_HandSolder, symbol Device:R_US
- J4: value Barrel_Jack_Switch_Pin3Ring -> 12V
Connections:
- net +3.3V: now also C2.1, J10.1 (Pin_1), J7.1 (Pin_1), R16.1, R17.1, R19.1, R20.1
- net +5V: now also J8.1 (Pin_1)
- net AC: now also F1.1; no longer F1.2
- net ADC1_CH7: now also J10.10 (Pin_10)
- net GND: now also C2.2, J10.2 (Pin_2), J7.2 (Pin_2), J8.2 (Pin_2), J9.2 (Pin_2)
- net I2C_SCL: now also J7.6 (Pin_6)
- net I2C_SDA: now also J7.5 (Pin_5)
- net IN1: now also J10.6 (Pin_6)
- net IN2: now also J10.5 (Pin_5)
- net IN3: now also J10.4 (Pin_4)
- net IN4: now also J7.10 (Pin_10)
- net IO0: now also J8.3 (Pin_3)
- net IO2: now also J8.5 (Pin_5)
- net LCD_DC: now also J10.8 (Pin_8)
- net LCD_RST: now also J10.7 (Pin_7)
- net MTCK: now also J8.10 (Pin_10)
- net MTDI: now also J8.9 (Pin_9)
- net MTDO: now also J7.4 (Pin_4)
- net MTMS: now also J7.3 (Pin_3)
- net PT100: now also J10.9 (Pin_9)
- net RXD: now also J8.4 (Pin_4)
- net SSRIN1: now also J8.7 (Pin_7)
- net SSRIN2: now also J7.9 (Pin_9)
- net TXD: now also J8.6 (Pin_6)
- net VSPI_CLK: now also J7.7 (Pin_7)
- net VSPI_CS0: now also J8.8 (Pin_8)
- net VSPI_D: now also J10.3 (Pin_3)
- net VSPI_Q: now also J7.8 (Pin_8)
- net at R32.2, SW7.2: now also R20.2
- net at K1.2 (L2): now also F1.2; no longer F1.1
- net +12V: now reaches C6.1, J4.1, U4.1 (IN)
- net +12V: now also J9.1 (Pin_1)
- net at R30.2, SW4.2: now also R17.2
- net at R31.2, SW5.2: now also R19.2
- net at R29.2, SW6.2: now also R16.2
- no-connect marks 23 -> 19
Other:
- note added: "DISPLAY"
- note added: "ESP32 WROOM"
- note added: "JTAG 10PIN"
- note added: "JTAG Debugging, With OpenOCD https://docs.espressif.com/projects/esp-idf/en/ latest/esp32/api-guides/jtag-debugging/index.html"
- note added: "PINOUT"
- note added: "PT100-PREAMP"
- note added: "Pinout Image https://electropeak.com/learn/wp-content/uploads/2021/02/ 1-3-Inch-240x240-IPS-SPI-HD-LCD-Full-Color-Display-OLED-Module-Pin.jpg"
- note added: "SSR OUTPUT"
- note added: "SUPPLY VOLTAGE"
- note added: "USB2SERIAL"
- note removed: "JTAG Debugging, With OpenOCD https://docs.espressif.com/projects/esp-idf/en/latest/esp32/api-guides/jtag-debugging/index.html"
- note removed: "Need To Add External Pull Up"
- note removed: "OLED 0.91Inch"
- note removed: "Omron SSR G3MB-202P"
- note removed: "PT100/RTD Signal Conditioning"
- note removed: "Pinout Image https://electropeak.com/learn/wp-content/uploads/2021/02/1-3-Inch-240x240-IPS-SPI-HD-LCD-Full-Color-Display-OLED-Module-Pin.jpg"
- note removed: "Todo List: 1. make PT100(RTD) signal conditioning based on microchip's appnote AN 687 2. make esp32/esp8266 connection 3. make control input connection 4. make color display or oled for UI There is some Information about SSR type by omron on their catalog manual page 15"
- note removed: "Voltage Regulator"
- note removed: "wemos d1"
- company: (none) -> AHAH TERROR
- moved on the sheet: C1, C10, C11, C12, C13, C14, C15, C16, C17, C18, C19, C3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

Commit message: [6-7-1245] finish first layout, need to review
Parts:
- removed D6: 3.3VPWR, LED_THT:LED_D5.0mm, symbol Device:LED
- removed H3: MountingHole_Pad, MountingHole:MountingHole_3.2mm_M3_DIN965_Pad, symbol Mechanical:MountingHole_Pad
- removed J1: AC_Con1, TerminalBlock_MetzConnect:TerminalBlock_MetzConnect_Type011_RT05502HBWC_1x02_P5.00mm_Horizontal, symbol Connector:Screw_Terminal_01x02
- removed J11: JTAG10, Connector_IDC:IDC-Header_2x10_P2.54mm_Vertical, symbol Connector:Conn_ARM_JTAG_SWD_10
- removed R11: 1k, Resistor_SMD:R_0805_2012Metric_Pad1.20x1.40mm_HandSolder, symbol Device:R_US
- added J1: ACCON, TerminalBlock_MetzConnect:TerminalBlock_MetzConnect_Type055_RT01503HDWU_1x03_P5.00mm_Horizontal, symbol Connector:Screw_Terminal_01x03
- added J13: JTAG10, Connector_PinHeader_2.54mm:PinHeader_2x05_P2.54mm_Vertical, symbol Connector:Conn_ARM_JTAG_SWD_10
- C1, C10, C11, C12, C13, C14, C15, C16, C17, C18, C19, C2, C3, C8, C9: footprint Capacitor_THT:C_Disc_D4.3mm_W1.9mm_P5.00mm -> Capacitor_SMD:C_1206_3216Metric_Pad1.33x1.80mm_HandSolder
- C6, C7: footprint Capacitor_THT:CP_Radial_D6.3mm_P2.50mm -> Capacitor_SMD:C_1206_3216Metric_Pad1.33x1.80mm_HandSolder
- D1, D4: footprint Diode_THT:D_DO-41_SOD81_P10.16mm_Horizontal -> Diode_SMD:D_SOD-123
- D2, D3, D5, D7, D8: footprint LED_THT:LED_D5.0mm -> LED_SMD:LED_2010_5025Metric_Pad1.52x2.65mm_HandSolder
- J6: footprint (none) -> Connector_USB:USB_B_OST_USB-B1HSxx_Horizontal
- SW2, SW3, SW4, SW5, SW6, SW7: footprint (none) -> Button_Switch_SMD:SW_SPST_B3S-1000
- renumbered RA to RA1, RB to RB1
Connections:
- net +3.3V: now also J13.1 (VTref)
- net AC: now also J1.1 (Pin_1)
- net EN: now also J13.10 (~{RESET})
- net GND: now also J13.3 (GND), J13.5 (GND), J13.9 (GNDDetect)
- net MTCK: now also J13.4 (SWCLK/TCK)
- net MTDI: now also J13.8 (NC/TDI)
- net MTDO: now also J13.6 (SWO/TDO)
- net MTMS: now also J13.2 (SWDIO/TMS)
- net at K1.1 (L1): now also J1.3 (Pin_3)
Other:
- moved on the sheet: C19, D7, D8, H1, H2, H4, H5, R26, R27, R32, SW7

Commit message: [8-06-0716] finish up layout plus adding several random graphic
Parts:
- removed J12: ST7789, Connector_PinSocket_2.54mm:PinSocket_1x07_P2.54mm_Vertical, symbol Connector_Generic:Conn_01x07
- added J11: ST7789, Connector_PinSocket_2.54mm:PinSocket_1x08_P2.54mm_Vertical, symbol Connector_Generic:Conn_01x08
- C1, C10, C11, C12, C13, C14, C15, C16, C17, C18, C19, C2, C3, C6, C7, C8, C9: footprint Capacitor_SMD:C_1206_3216Metric_Pad1.33x1.80mm_HandSolder -> Capacitor_SMD:C_0805_2012Metric_Pad1.18x1.45mm_HandSolder
- D2, D3, D5, D7, D8: footprint LED_SMD:LED_2010_5025Metric_Pad1.52x2.65mm_HandSolder -> LED_SMD:LED_1206_3216Metric_Pad1.42x1.75mm_HandSolder
- J1: footprint TerminalBlock_MetzConnect:TerminalBlock_MetzConnect_Type055_RT01503HDWU_1x03_P5.00mm_Horizontal -> TerminalBlock_Phoenix:TerminalBlock_Phoenix_PT-1,5-3-5.0-H_1x03_P5.00mm_Horizontal
- J3, J5, J9: footprint TerminalBlock_MetzConnect:TerminalBlock_MetzConnect_Type011_RT05502HBWC_1x02_P5.00mm_Horizontal -> TerminalBlock_Phoenix:TerminalBlock_Phoenix_PT-1,5-2-5.0-H_1x02_P5.00mm_Horizontal
- SW2, SW3: footprint Button_Switch_SMD:SW_SPST_B3S-1000 -> Button_Switch_SMD:SW_Push_1P1T_NO_6x6mm_H9.5mm
- SW4: value IO0 -> D; footprint Button_Switch_SMD:SW_SPST_B3S-1000 -> Button_Switch_SMD:SW_Push_1P1T_NO_6x6mm_H9.5mm
- SW5: value IO0 -> U; footprint Button_Switch_SMD:SW_SPST_B3S-1000 -> Button_Switch_SMD:SW_Push_1P1T_NO_6x6mm_H9.5mm
- SW6: value IO0 -> L; footprint Button_Switch_SMD:SW_SPST_B3S-1000 -> Button_Switch_SMD:SW_Push_1P1T_NO_6x6mm_H9.5mm
- SW7: value IO0 -> R; footprint Button_Switch_SMD:SW_SPST_B3S-1000 -> Button_Switch_SMD:SW_Push_1P1T_NO_6x6mm_H9.5mm
Connections:
- net +3.3V: now also J11.2 (Pin_2), J11.8 (Pin_8)
- net GND: now also J11.1 (Pin_1)
- net LCD_DC: now also J11.6 (Pin_6)
- net LCD_RST: now also J11.5 (Pin_5)
- net VSPI_CLK: now also J11.3 (Pin_3)
- net VSPI_D: now also J11.4 (Pin_4)
- net IO2 renamed LCD_CS
- net LCD_CS: now also J11.7 (Pin_7)
Other:
- moved on the sheet: C6, C7, C8, C9, D7, D8, J4, J9, R26, R27, U3, U4
