File: hardware/v2/solder-reflow.kicad_sch (KiCad schematic)
At the start: 91 parts, among them J1 ACCON, J10 PINOUT, J11 ST7789, J13 JTAG10, J2 OLED 0.91, J3 PTC_Con, J4 12V, J5 SSROUT2, J6 USB_B, J7 PINOUT, J8 PINOUT, J9 12VIN, K1 G3MB202PDC12, Q1 SS8550, Q2 SS8550, Q3 SS8050, Q4 SS8050, SW2 RST, SW3 IO0, SW4 D, SW5 U, SW6 L, SW7 R, U1 TL431LP, U2 TL074, U3 AMS1117-3.3, U4 L7805, U6 ESP32-WROOM-32D, U7 CH340C

Commit message: feat: start creating schematic with esp32-s3 soc
Parts:
- removed D8: RXD, LED_SMD:LED_1206_3216Metric_Pad1.42x1.75mm_HandSolder, symbol Device:LED
- removed J6: USB_B, Connector_USB:USB_B_OST_USB-B1HSxx_Horizontal, symbol Connector:USB_B
- removed Q3, Q4: SS8050, Package_TO_SOT_SMD:SOT-23_Handsoldering, symbol Transistor_BJT:BC817
- removed R10, R7: 10k, Resistor_SMD:R_0805_2012Metric_Pad1.20x1.40mm_HandSolder, symbol Device:R_US
- removed U2: TL074, Package_SO:SOIC-14_3.9x8.7mm_P1.27mm, symbol Amplifier_Operational:TL074
- removed U3: AMS1117-3.3, Package_TO_SOT_SMD:SOT-223-3_TabPin2, symbol Regulator_Linear:AMS1117-3.3
- removed U4: L7805, Package_TO_SOT_THT:TO-220F-3_Horizontal_TabDown, symbol Regulator_Linear:L7805
- removed U7: CH340C, Package_SO:SOIC-16_3.9x9.9mm_P1.27mm, symbol Interface_USB:CH340C
- added C20: 100uF/16V, Capacitor_SMD:C_0805_2012Metric_Pad1.18x1.45mm_HandSolder, symbol Device:C_Polarized
- added C21: 100nF, Capacitor_SMD:C_0805_2012Metric_Pad1.18x1.45mm_HandSolder, symbol Device:C
- added C22: 22uF, Capacitor_SMD:C_0805_2012Metric_Pad1.18x1.45mm_HandSolder, symbol Device:C
- added C23, C5: 1uF, Capacitor_SMD:C_0805_2012Metric_Pad1.18x1.45mm_HandSolder, symbol Device:C
- added D6: TXD, LED_SMD:LED_1206_3216Metric_Pad1.42x1.75mm_HandSolder, symbol Device:LED
- added F2: Fuse, Fuse:Fuseholder_Littelfuse_100_series_5x30mm, symbol Device:Fuse
- added J12: USB_C_Receptacle_USB2.0_14P, symbol Connector:USB_C_Receptacle_USB2.0_14P
- added J14: 220V, TerminalBlock_Phoenix:TerminalBlock_Phoenix_PT-1,5-2-5.0-H_1x02_P5.00mm_Horizontal, symbol Connector:Screw_Terminal_01x02
- added J6: InputButton, Connector_PinSocket_2.54mm:PinSocket_1x08_P2.54mm_Vertical, symbol Connector_Generic:Conn_01x08
- added PS1: HLK-2M12 12V 2W, Converter_ACDC:Converter_ACDC_Hi-Link_HLK-2Mxx, symbol Converter_ACDC:HLK-2M12
- added R11, R21: 5K1, Resistor_SMD:R_0805_2012Metric_Pad1.20x1.40mm_HandSolder, symbol Device:R_US
- added R33, R35, R39, R41: 10k, Resistor_SMD:R_0805_2012Metric_Pad1.20x1.40mm_HandSolder, symbol Device:R_US
- added R34, R36, R40: 22k, Resistor_SMD:R_0805_2012Metric_Pad1.20x1.40mm_HandSolder, symbol Device:R_US
- added R37, R38: 10k, Resistor_THT:R_Axial_DIN0309_L9.0mm_D3.2mm_P15.24mm_Horizontal, symbol Device:R_US
- added R42: 1k, Resistor_SMD:R_0805_2012Metric_Pad1.20x1.40mm_HandSolder, symbol Device:R_US
- added SW1, SW8: R, Button_Switch_SMD:SW_Push_1P1T_NO_6x6mm_H9.5mm, symbol Switch:SW_Push
- added SW9: Boot, Button_Switch_SMD:SW_Push_1P1T_NO_6x6mm_H9.5mm, symbol Switch:SW_Push
- added U2, U9: LM324, Package_SO:SOIC-14_3.9x8.7mm_P1.27mm, symbol Amplifier_Operational:LM324
- added U3: L7805, Package_TO_SOT_THT:TO-220F-3_Horizontal_TabDown, symbol Regulator_Linear:L7805
- added U4: AMS1117-3.3, Package_TO_SOT_SMD:SOT-223-3_TabPin2, symbol Regulator_Linear:AMS1117-3.3
- added U5: ESP32-S3-WROOM-1, RF_Module:ESP32-S3-WROOM-1U, symbol RF_Module:ESP32-S3-WROOM-1
- added U8: H11AA1, Package_DIP:DIP-6_W7.62mm_SMDSocket_SmallPads, symbol Isolator:H11AA1
- C10, C11: value 100nF -> 1uF
- D7: value TXD -> RXD
- SW3: value IO0 -> R
Connections:
- net +12V: now also C20.1, PS1.4 (+Vout), U3.1 (IN)
- net +3.3V: now also C21.1, C22.1, C23.1, J6.7 (Pin_7), R33.1, R35.1, R39.1, R41.1, R42.1, U4.2 (VO), U5.2 (3V3); no longer C10.1
- net +5V: now also J12.A4 (VBUS), J12.A9 (VBUS), J12.B4 (VBUS), J12.B9 (VBUS), U2.4 (V+), U3.3 (OUT), U4.3 (VI)
- net AC: now also F2.1, PS1.1 (AC/L)
- net EN: now also U5.3 (EN); no longer C11.1, U6.3 (EN)
- net GND: now also C20.2, C21.2, C22.2, C23.2, C5.2, J12.A1 (GND), J12.A12 (GND), J12.B1 (GND), J12.B12 (GND), J6.8 (Pin_8), PS1.3 (-Vout), R11.1, R21.1, SW1.1, SW8.1, SW9.1, U2.11 (V-), U3.2 (GND), U4.1 (GND), U5.1 (GND), U5.40 (GND), U5.41 (GND), U8.4
- net IN1: now also U5.8 (IO15)
- net IN2: now also U5.9 (IO16)
- net IN3: now also U5.16 (IO46)
- net IN4: now also U5.10 (IO17)
- net IO0: now also R42.2, SW9.2, U5.27 (IO0); no longer SW3.2
- net MTCK: now also U5.32 (IO39)
- net MTDI: now also U5.34 (IO41)
- net MTDO: now also U5.33 (IO40)
- net MTMS: now also U5.35 (IO42)
- net PT100: now also U9.13 (-), U9.14
- net PT100Voltage: now also U9.5 (+)
- net RXD: now also D7.1 (K)
- net TXD: now also D6.1 (K); no longer D7.1 (K)
- net at RA1.1, RB1.2: now also U9.9 (-)
- net at C1.1, RA1.2: now also U9.12 (+), U9.8
- net sw4: now reaches R20.2, R32.2, SW7.2
- net sw4: now also J6.4 (Pin_4)
- net at R3.2, R6.1: now also U9.1
- net at R5.2, R6.2: now also U9.2 (-)
- net at R2.2, R4.1: now also U9.3 (+)
- net at C3.1, R9.1: now also U9.10 (+)
- net at D7.2 (A): now also R27.2; no longer R26.2
- net sw2: now reaches R17.2, R30.2, SW4.2
- net sw2: now also J6.2 (Pin_2)
- net at R4.2: now also U9.6 (-), U9.7
- net sw3: now reaches R19.2, R31.2, SW5.2
- net sw3: now also J6.3 (Pin_3)
- net sw1: now reaches R16.2, R29.2, SW6.2
- net sw1: now also J6.1 (Pin_1)
- new net: F2.2, J14.1 (Pin_1), R38.1
- new net: J14.2 (Pin_2), PS1.2 (AC/N), R37.1
- new net: R39.2, R40.2, SW3.2
- new net: C11.1, R40.1, U8.6
- new net: R37.2, U8.1
- new net: D6.2 (A), R26.2
- new net: R38.2, U8.2
- new net: J12.B5 (CC2), R21.2
- new net: J12.A5 (CC1), R11.2
- new net IN5: C5.1, R34.1, U5.11 (IO18)
- new net IN6: C10.1, R36.1, U5.23 (IO21)
- new net RXD0: U5.36 (RXD0)
- new net TXD0: U5.37 (TXD0)
- new net USB_D+: J12.A7 (D-), J12.B7 (D-), U5.14 (IO20)
- new net USB_D-: J12.A6 (D+), J12.B6 (D+), U5.13 (IO19)
- new net ZC_INPUT: R41.2, U5.15 (IO3), U8.5
- new net sw5: J6.5 (Pin_5), R33.2, R34.2, SW1.2
- new net sw6: J6.6 (Pin_6), R35.2, R36.2, SW8.2
- no-connect marks 19 -> 12
Other:
- note added: "Flash Using USB For the ESP32-S3, the USB peripheral is available, allowing you to flash the binaries without the need for an external USB-to-UART bridge. The USB on the ESP32-S3 uses the GPIO20 for D+ and GPIO19 for D-. If you are flashing for the first time, you need to get the ESP32-S3 into the download mode manually. To do so, press and hold the BOOT button and then press the RESET button onc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"
- note added: "TODO List: 1. change pt 100 signal conditioning to work with esp32 adc max voltage 2. add zero crossing reader with 15k resistor (look at minimum led current to be turned on) 3. Recheck IO pin if it equal and correct usage with old esp32 4. separate schematic into 2 region (low and high) 5. make pcb into breakable region (low and high) 6. use easy to connect connector for low and high region 7. t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"
- note removed: "USB2SERIAL"
- moved on the sheet: C14, C16, C17, C18, C19, D1, D2, D3, D4, D5, F1, J1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

Commit message: feat: finish basic schematic, need to re-check
Update README.md
Parts:
- removed C2, C23: 1uF, Capacitor_SMD:C_0805_2012Metric_Pad1.18x1.45mm_HandSolder, symbol Device:C
- removed C20: 100uF/16V, Capacitor_SMD:C_0805_2012Metric_Pad1.18x1.45mm_HandSolder, symbol Device:C_Polarized
- removed C21: 100nF, Capacitor_SMD:C_0805_2012Metric_Pad1.18x1.45mm_HandSolder, symbol Device:C
- removed C22: 22uF, Capacitor_SMD:C_0805_2012Metric_Pad1.18x1.45mm_HandSolder, symbol Device:C
- removed C7: 0.1uF, Capacitor_SMD:C_0805_2012Metric_Pad1.18x1.45mm_HandSolder, symbol Device:C_Polarized
- removed D2: SSR1, LED_SMD:LED_1206_3216Metric_Pad1.42x1.75mm_HandSolder, symbol Device:LED
- removed D4: 1N4001, Diode_SMD:D_SOD-123, symbol Diode:1N4001
- removed F2: Fuse, Fuse:Fuseholder_Littelfuse_100_series_5x30mm, symbol Device:Fuse
- removed H5: MountingHole_Pad, MountingHole:MountingHole_3.2mm_M3_DIN965_Pad, symbol Mechanical:MountingHole_Pad
- removed J1: ACCON, TerminalBlock_Phoenix:TerminalBlock_Phoenix_PT-1,5-3-5.0-H_1x03_P5.00mm_Horizontal, symbol Connector:Screw_Terminal_01x03
- removed J11: ST7789, Connector_PinSocket_2.54mm:PinSocket_1x08_P2.54mm_Vertical, symbol Connector_Generic:Conn_01x08
- removed J12: USB_C_Receptacle_USB2.0_14P, symbol Connector:USB_C_Receptacle_USB2.0_14P
- removed J13: JTAG10, Connector_PinHeader_2.54mm:PinHeader_2x05_P2.54mm_Vertical, symbol Connector:Conn_ARM_JTAG_SWD_10
- removed J2: OLED 0.91, Connector_PinHeader_2.54mm:PinHeader_1x04_P2.54mm_Vertical, symbol Connector:Conn_01x04_Pin
- removed J4: 12V, Connector_BarrelJack:BarrelJack_Horizontal, symbol Connector:Barrel_Jack_Switch_Pin3Ring
- removed RA1, RB1: 25k, Resistor_SMD:R_0805_2012Metric_Pad1.20x1.40mm_HandSolder, symbol Device:R_US
- removed U6: ESP32-WROOM-32D, RF_Module:ESP32-WROOM-32D, symbol RF_Module:ESP32-WROOM-32D
- removed U8: H11AA1, Package_DIP:DIP-6_W7.62mm_SMDSocket_SmallPads, symbol Isolator:H11AA1
- removed U9: LM324, Package_SO:SOIC-14_3.9x8.7mm_P1.27mm, symbol Amplifier_Operational:LM324
- added C2: 100uF/16V, Capacitor_SMD:C_0805_2012Metric_Pad1.18x1.45mm_HandSolder, symbol Device:C_Polarized
- added C4: 0.33uF, Capacitor_SMD:C_0805_2012Metric_Pad1.18x1.45mm_HandSolder, symbol Device:C_Polarized
- added C7: 22uF, Capacitor_SMD:C_0805_2012Metric_Pad1.18x1.45mm_HandSolder, symbol Device:C
- added D2: 1N4001, Diode_SMD:D_SOD-123, symbol Diode:1N4001
- added D4: SSR2, LED_SMD:LED_1206_3216Metric_Pad1.42x1.75mm_HandSolder, symbol Device:LED
- added H3: MountingHole_Pad, MountingHole:MountingHole_3.2mm_M3_DIN965_Pad, symbol Mechanical:MountingHole_Pad
- added J1: USB_C_Receptacle_USB2.0_14P, symbol Connector:USB_C_Receptacle_USB2.0_14P
- added J11: I2C, Connector_Molex:Molex_SL_171971-0004_1x04_P2.54mm_Vertical, symbol Connector_Generic:Conn_01x04
- added J12: JTAG10, Connector_PinHeader_2.54mm:PinHeader_2x05_P2.54mm_Vertical, symbol Connector:Conn_ARM_JTAG_SWD_10
- added J13: 12V, Connector_BarrelJack:BarrelJack_Horizontal, symbol Connector:Barrel_Jack_Switch_Pin3Ring
- added J15: LCD_CONN, Connector_Molex:Molex_SL_171971-0010_1x10_P2.54mm_Vertical, symbol Connector_Generic:Conn_01x10
- added J16: UART, Connector_Molex:Molex_SL_171971-0004_1x04_P2.54mm_Vertical, symbol Connector_Generic:Conn_01x04
- added J2: I2S, Connector_Molex:Molex_SL_171971-0006_1x06_P2.54mm_Vertical, symbol Connector_Generic:Conn_01x06
- added J4: 220V, TerminalBlock_Phoenix:TerminalBlock_Phoenix_PT-1,5-2-5.0-H_1x02_P5.00mm_Horizontal, symbol Connector:Screw_Terminal_01x02
- added JP1: InH11AA1, Jumper:SolderJumper-2_P1.3mm_Open_TrianglePad1.0x1.5mm, symbol Jumper:SolderJumper_2_Open
- added R10, R7: 4K7, Resistor_SMD:R_0805_2012Metric_Pad1.20x1.40mm_HandSolder, symbol Device:R_US
- added unit 1 of U2
- added unit 4 of U2
- added unit 3 of U2
- added unit 2 of U2
- added U6: 74LS14, Package_DIP:DIP-14_W7.62mm_SMDSocket_SmallPads, symbol 74xx:74LS14
- added U7: H11AA1, Package_DIP:DIP-6_W7.62mm_SMDSocket_SmallPads, symbol Isolator:H11AA1
- C1, C3: value 1nF -> 10nF
- C11: value 1uF -> 22uF
- C12: value 100nF -> 1uF
- C13, C8, C9: value 22uF -> 1uF
- C15: value 100nF -> 22uF
- C17, C18: value 1uF -> 100nF
- C6: value 0.33uF -> 0.1uF
- D3: value POWER_LED -> TXD
- D5: value SSR2 -> SSR1
- D6: value TXD -> RXD
- D7: value RXD -> POWER_LED
- J14: value 220V -> SSROUT2
- J5: value SSROUT2 -> HEATER
- R12: value 4K7 -> 9K1
- R13: value 4K7 -> 1K
- R18, R27: value 1k -> 10k
- R20, R35: value 10k -> 22k
- R24: value 10k -> 1k
- R31, R32: value 22k -> 10k
- R37: value 10k -> 22k; footprint Resistor_THT:R_Axial_DIN0309_L9.0mm_D3.2mm_P15.24mm_Horizontal -> Resistor_SMD:R_0805_2012Metric_Pad1.20x1.40mm_HandSolder
- R38: value 10k -> 1k; footprint Resistor_THT:R_Axial_DIN0309_L9.0mm_D3.2mm_P15.24mm_Horizontal -> Resistor_SMD:R_0805_2012Metric_Pad1.20x1.40mm_HandSolder
- R40: value 22k -> 10k; footprint Resistor_SMD:R_0805_2012Metric_Pad1.20x1.40mm_HandSolder -> Resistor_THT:R_Axial_DIN0309_L9.0mm_D3.2mm_P15.24mm_Horizontal
- R41: footprint Resistor_SMD:R_0805_2012Metric_Pad1.20x1.40mm_HandSolder -> Resistor_THT:R_Axial_DIN0309_L9.0mm_D3.2mm_P15.24mm_Horizontal
- SW1: value R -> L
- SW3: value R -> SWH11AA1
- SW6: value L -> R
Connections:
- net ADC1_CH7 is gone; now on net CS0: J10.10 (Pin_10)
- net LCD_CS is gone; now on net MTDI: J8.5 (Pin_5)
- net LCD_DC is gone; now on net IO8: J10.8 (Pin_8)
- net LCD_RST is gone; now on net I2C_SCL: J10.7 (Pin_7)
- net VSPI_CLK is gone; now on net TXD0: J7.7 (Pin_7)
- net VSPI_CS0 is gone; now on net IN3: J8.8 (Pin_8)
- net VSPI_D is gone; now on net ZC_INPUT: J10.3 (Pin_3)
- net VSPI_Q is gone; now on net RXD0: J7.8 (Pin_8)
- net +12V: now also C2.1, C4.1, J13.1; no longer C6.1
- net +3.3V: now also C11.1, C14.1, C15.1, C16.1, R22.1, R31.1, R32.1, J11.1 (Pin_1), J12.1 (VTref), J15.2 (Pin_2), J16.1 (Pin_1), J2.1 (Pin_1), R10.2, R7.2; no longer C12.1, C13.1, C9.1, J10.1 (Pin_1), J7.1 (Pin_1), R12.2, R13.2, R20.1, R35.1, R41.1
- net +5V: now also C6.1, R38.2, C7.1, D2.2 (A), J1.A4 (VBUS), J1.A9 (VBUS), J1.B4 (VBUS), J1.B9 (VBUS), J15.3 (Pin_3), U6.14 (VCC); no longer C8.1, J8.1 (Pin_1), R22.2
- net EN: now also C17.1, J12.10 (~{RESET}); no longer C14.1
- net GND: now also D7.1 (K), J14.2 (Pin_2), R13.2, C2.2, C4.2, C7.2, D4.1 (K), J1.A1 (GND), J1.A12 (GND), J1.B1 (GND), J1.B12 (GND), J11.4 (Pin_4), J12.3 (GND), J12.5 (GND), J12.9 (GNDDetect), J13.2, J13.3, J15.1 (Pin_1), J16.4 (Pin_4), J2.6 (Pin_6), U6.7 (GND), U7.4; no longer D3.1 (K), J10.2 (Pin_2), J5.2 (Pin_2), J7.2 (Pin_2), J8.2 (Pin_2)
- net I2C_SCL: now also U5.7 (IO7), J11.3 (Pin_3), R10.1; no longer J7.6 (Pin_6), R13.1
- net I2C_SDA: now also J10.6 (Pin_6), U5.6 (IO6), J11.2 (Pin_2), R7.1; no longer J7.5 (Pin_5), R12.1
- net IN1: now also C5.1, J7.5 (Pin_5), R20.1; no longer C18.1, J10.6 (Pin_6), R29.1
- net IN2: now also C8.1, J7.6 (Pin_6), R29.1; no longer C16.1, J10.5 (Pin_5), R30.1
- net IN3: now also C9.1, R30.1; no longer C17.1, J10.4 (Pin_4), R31.1
- net IN4: now also C10.1, J7.9 (Pin_9), R34.1; no longer C19.1, J7.10 (Pin_10), R32.1
- net IN5: now also C12.1, J7.10 (Pin_10), R35.1; no longer C5.1, R34.1
- net IN6: now also C13.1, J8.1 (Pin_1); no longer C10.1
- net IO0: now also C18.1; no longer C15.1, J8.3 (Pin_3)
- net MTCK: now also J8.3 (Pin_3), J12.4 (SWCLK/TCK); no longer J8.10 (Pin_10)
- net MTDI: now also J12.8 (NC/TDI); no longer J8.9 (Pin_9)
- net MTDO: now also J8.4 (Pin_4), J12.6 (SWO/TDO); no longer J7.4 (Pin_4)
- net MTMS: now also J8.6 (Pin_6), J12.2 (SWDIO/TMS); no longer J7.3 (Pin_3)
- net PT100: now also J10.4 (Pin_4), R12.1, U5.4 (IO4), U2.14; no longer J10.9 (Pin_9)
- net PT100Voltage: now also U2.5 (+)
- net RXD: now also D6.1 (K); no longer D7.1 (K), J8.4 (Pin_4)
- net RXD0: now also J16.3 (Pin_3)
- net SSRIN1: now also J10.1 (Pin_1), R23.1, U5.39 (IO1); no longer J8.7 (Pin_7), R15.1
- net SSRIN2: now also J10.2 (Pin_2), R18.1, U5.38 (IO2); no longer J7.9 (Pin_9), R23.1
- net TXD: now also D3.1 (K); no longer D6.1 (K), J8.6 (Pin_6)
- net TXD0: now also J16.2 (Pin_2)
- net USB_D+: now also J1.A7 (D-), J1.B7 (D-)
- net USB_D-: now also J1.A6 (D+), J1.B6 (D+)
- net ZC_INPUT: now also U6.2; no longer R41.2
- net sw1: now also R20.2, SW1.2; no longer R29.2, SW6.2
- net sw2: now also R29.2; no longer R30.2
- net sw3: now also R30.2; no longer R31.2
- net sw4: now also R31.2, R34.2, SW6.2; no longer R20.2, R32.2, SW7.2
- net sw5: now also R32.2, R35.2, SW7.2; no longer R33.2, R34.2, SW1.2
- net sw6: now also R33.2; no longer R35.2
- net at R24.2: now also J14.1 (Pin_1), Q1.3 (C); no longer Q2.2 (E)
- net at C1.1: now also U2.12 (+), U2.8, U2.9 (-)
- net at K1.1 (L1): now also J5.2 (Pin_2)
- net at R5.2, R6.2: now also U2.2 (-)
- net at F1.2: now also R41.1, J4.1 (Pin_1); no longer K1.2 (L2)
- net at C3.1, R9.1: now also U2.10 (+)
- net IO8: now reaches U5.12 (IO8)
- net IO8: now also J15.10 (Pin_10)
- net QUADHD: now reaches U5.17 (IO9)
- net QUADHD: now also J10.9 (Pin_9), J15.7 (Pin_7)
- net CS0: now reaches U5.18 (IO10)
- net CS0: now also J15.9 (Pin_9)
- net MOSI: now reaches U5.19 (IO11)
- net MOSI: now also J7.1 (Pin_1), J15.4 (Pin_4)
- net SCLK: now reaches U5.20 (IO12)
- net SCLK: now also J7.2 (Pin_2), J15.5 (Pin_5)
- net MISO: now reaches U5.21 (IO13)
- net MISO: now also J7.3 (Pin_3), J15.6 (Pin_6)
- net QUADWP: now reaches U5.22 (IO14)
- net QUADWP: now also J7.4 (Pin_4), J15.8 (Pin_8)
- net WS: now reaches U5.24 (IO47)
- net WS: now also J8.9 (Pin_9), J2.4 (Pin_4)
- net DIO: now reaches U5.25 (IO48)
- net DIO: now also J8.10 (Pin_10), J2.5 (Pin_5)
- net BCLK: now reaches U5.26 (IO45)
- net BCLK: now also J8.7 (Pin_7), J2.3 (Pin_3)
- net MCLK: now reaches U5.31 (IO38)
- net MCLK: now also J8.2 (Pin_2), J2.2 (Pin_2)
- net IO5: now reaches U5.5 (IO5)
- net IO5: now also J10.5 (Pin_5)
- net at R3.2, R6.1: now also U2.1
- net at R2.2, R4.1: now also U2.3 (+)
- net at R38.1: now also D7.2 (A); no longer J14.1 (Pin_1)
- net NEUT: now reaches R40.1
- net NEUT: now also K1.2 (L2), PS1.2 (AC/N), J4.2 (Pin_2); no longer C11.1
- net at R27.2: now also R37.2, SW3.2; no longer D7.2 (A)
- net at D3.2 (A): now also R22.2; no longer R22.1
- net at R4.2: now also U2.6 (-), U2.7
- net at Q2.1 (B), R23.2: now also R15.1; no longer R24.1
- net at Q2.3 (C), R25.2: now also K1.3 (+); no longer J5.1 (Pin_1)
- net at Q1.1 (B), R14.1: now also R18.2; no longer R15.2
- net at R21.2: now also J1.B5 (CC2)
- net at R11.2: now also J1.A5 (CC1)
- net AC renamed LINE
- net LINE: now also J5.1 (Pin_1)
- new net: R40.2, U7.1
- new net: R41.2, U7.2
- new net: R39.2, U6.1, U7.5
- new net: JP1.2 (B), U7.6
- new net: R12.2, R13.1, U2.13 (-)
- new net: C19.1, JP1.1 (A), R37.1
- new net: D4.2 (A), R24.1
- new net: D2.1 (K), Q2.2 (E), R15.2
- no-connect marks 12 -> 8
Other:
- note added: "AC SUPPLY VOLTAGE"
- note added: "DC SUPPLY VOLTAGE"
- note added: "ESP32-S3"
- note added: "Gain = 1 + (9,1K / 1K) = 10.1"
- note added: "I2C"
- note added: "I2S"
- note added: "JTAG"
- note added: "LCD"
- note added: "Reference Design Schematic: esp32-s3 https://docs.espressif.com/projects/esp-hardware-design-guidelines/en/latest/esp32s3/esp-hardware-design-guidelines-en-master-esp32s3.pdf"
- note added: "SSR"
- note added: "TODO List: 1. change pt 100 signal conditioning to work with esp32 adc max voltage 2. add zero crossing reader with 15k resistor (look at minimum led current to be turned on) 3. Recheck IO pin if it equal and correct usage with old esp32 4. separate schematic into 2 region (low and high) 5. make pcb into breakable region (low and high) 6. use easy to connect connector for low and high region make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"
- note added: "Target Temp for PT100 is Less 400*C, Based on Resistance table its about 250ohm current source is 1mA, with tolerance, if resistance of PT100 300 ohm it will be 300mV, adding non inverting to increase gain into 3V (x10)"
- note added: "UART"
- note added: "USBC"
- note added: "if temp is not more than 400, voltage on pin 12 will never exeed 300mV"
- note added: "typical VOH = 3.4 https://www.ti.com/lit/ds/symlink/sn54ls14-sp.pdf?ts=1757765835115"
- note removed: "DISPLAY"
- note removed: "ESP32 WROOM"
- note removed: "JTAG 10PIN"
- note removed: "JTAG Debugging, With OpenOCD https://docs.espressif.com/projects/esp-idf/en/ latest/esp32/api-guides/jtag-debugging/index.html"
- note removed: "LCD_BACKLIGHT"
- note removed: "Pinout Image https://electropeak.com/learn/wp-content/uploads/2021/02/ 1-3-Inch-240x240-IPS-SPI-HD-LCD-Full-Color-Display-OLED-Module-Pin.jpg"
- note removed: "Pins SCK/CLK, SDO/SD0, SDI/SD1, SHD/SD2, SWP/SD3 and SCS/CMD, namely, GPIO6 to GPIO11 are connected to the integrated SPI flash integrated on the module and are not recommended for other uses."
- note removed: "Reference Design Schematic: ESP32-DevKit V4 https://dl.espressif.com/dl/schematics/esp32_devkitc_v4-sch.pdf"
- note removed: "SSR OUTPUT"
- note removed: "SUPPLY VOLTAGE"
- note removed: "TODO List: 1. change pt 100 signal conditioning to work with esp32 adc max voltage 2. add zero crossing reader with 15k resistor (look at minimum led current to be turned on) 3. Recheck IO pin if it equal and correct usage with old esp32 4. separate schematic into 2 region (low and high) 5. make pcb into breakable region (low and high) 6. use easy to connect connector for low and high region 7. t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"
- note removed: "Target Temp for PT100 is Less 400*C, Based on Resistance table its about 250ohm"
- moved on the sheet: J10

Commit message: feat: basic board layout finished
Parts:
- removed H3, H4: MountingHole_Pad, MountingHole:MountingHole_3.2mm_M3_DIN965_Pad, symbol Mechanical:MountingHole_Pad
- removed J13: 12V, Connector_BarrelJack:BarrelJack_Horizontal, symbol Connector:Barrel_Jack_Switch_Pin3Ring
- added C20: 100nF, Capacitor_SMD:C_0805_2012Metric_Pad1.18x1.45mm_HandSolder, symbol Device:C
- added J17: USB_C_Receptacle_USB2.0_14P, Connector_USB:USB_C_Receptacle_GCT_USB4110, symbol Connector:USB_C_Receptacle_USB2.0_14P
- added J18, J19: High_To_Low_Link, Connector_IDC:IDC-Header_2x05_P2.54mm_Vertical, symbol Connector_Generic:Conn_02x05_Odd_Even
- added Q3, Q4: SS8050, Package_TO_SOT_SMD:SOT-23_Handsoldering, symbol Transistor_BJT:BC817
- added R43, R44: 5K1, Resistor_SMD:R_0805_2012Metric_Pad1.20x1.40mm_HandSolder, symbol Device:R_US
- added R45, R46: 10k, Resistor_SMD:R_0805_2012Metric_Pad1.20x1.40mm_HandSolder, symbol Device:R_US
- added U8: CH340C, Package_SO:SOIC-16_3.9x9.9mm_P1.27mm, symbol Interface_USB:CH340C
- C2: footprint Capacitor_SMD:C_0805_2012Metric_Pad1.18x1.45mm_HandSolder -> Capacitor_THT:CP_Radial_D8.0mm_P3.50mm
- J1: footprint (none) -> Connector_USB:USB_C_Receptacle_GCT_USB4110
- J10, J7, J8: footprint Connector_PinHeader_2.54mm:PinHeader_1x10_P2.54mm_Vertical -> Connector_Molex:Molex_SL_171971-0010_1x10_P2.54mm_Vertical
- J12: footprint Connector_PinHeader_2.54mm:PinHeader_2x05_P2.54mm_Vertical -> Connector_IDC:IDC-Header_2x05_P2.54mm_Vertical
- J6: footprint Connector_PinSocket_2.54mm:PinSocket_1x08_P2.54mm_Vertical -> Connector_Molex:Molex_KK-254_AE-6410-08A_1x08_P2.54mm_Vertical
- R40, R41: value 10k -> 10k 1W
Connections:
- net RXD is gone; now on net RXD0: D6.1 (K)
- net TXD is gone; now on net TXD0: D3.1 (K)
- net +12V: now also J18.6 (Pin_6), J19.6 (Pin_6)
- net +3.3V: now also C20.1, J18.10 (Pin_10), J19.10 (Pin_10), U8.16 (VCC), U8.4 (V3)
- net +5V: now also J17.A4 (VBUS), J17.A9 (VBUS), J17.B4 (VBUS), J17.B9 (VBUS), J18.9 (Pin_9), J19.9 (Pin_9)
- net EN: now also Q3.3 (C)
- net GND: now also C20.2, J17.A1 (GND), J17.A12 (GND), J17.B1 (GND), J17.B12 (GND), J18.8 (Pin_8), J19.8 (Pin_8), R43.1, R44.1, U8.1 (GND)
- net IO0: now also Q4.3 (C)
- net LINE: now also R41.1, J18.1 (Pin_1), J19.1 (Pin_1)
- net NEUT: now also J18.5 (Pin_5), J19.5 (Pin_5)
- net RXD0: now also U8.2 (TXD)
- net SSRIN1: now also J18.2 (Pin_2), J19.2 (Pin_2)
- net SSRIN2: now also J18.4 (Pin_4), J19.4 (Pin_4)
- net TXD0: now also U8.3 (RXD)
- net ZC_INPUT: now also J18.7 (Pin_7), J19.7 (Pin_7)
- net at F1.2, J4.1 (Pin_1): no longer R41.1
- new net: Q4.1 (B), R46.1
- new net: J17.A5 (CC1), R43.2
- new net: J17.A6 (D+), J17.B6 (D+), U8.5 (UD+)
- new net: J17.A7 (D-), J17.B7 (D-), U8.6 (UD-)
- new net: J17.B5 (CC2), R44.2
- new net: Q3.1 (B), R45.1
- new net DTR: Q4.2 (E), R45.2, U8.13 (~{DTR})
- new net RTS: Q3.2 (E), R46.2, U8.14 (~{RTS})
- no-connect marks 8 -> 15
Other:
- note added: "High To Low Voltage Link"
- note added: "LM324 Vo=(1+R1/R2)*vref which: vref approx 2.5v R1=0 R2=~"
- note added: "Reference Design Schematic: esp32-s3 https://docs.espressif.com/projects/esp-hardware-design-guidelines/en/latest/esp32s3/esp-hardware-design-guidelines-en-master-esp32s3.pdf https://dl.espressif.com/dl/schematics/SCH_ESP32-S3-DevKitC-1_V1.1_20221130.pdf"
- note added: "UART to USB"
- note removed: "Reference Design Schematic: esp32-s3 https://docs.espressif.com/projects/esp-hardware-design-guidelines/en/latest/esp32s3/esp-hardware-design-guidelines-en-master-esp32s3.pdf"
- note removed: "TL431 Vo=(1+R1/R2)*vref which: vref approx 2.5v R1=0 R2=~"
- note removed: "TODO List: 1. change pt 100 signal conditioning to work with esp32 adc max voltage 2. add zero crossing reader with 15k resistor (look at minimum led current to be turned on) 3. Recheck IO pin if it equal and correct usage with old esp32 4. separate schematic into 2 region (low and high) 5. make pcb into breakable region (low and high) 6. use easy to connect connector for low and high region make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"
- company: AHAH TERROR -> CRUMBS Module
- title: Solder Reflow  -> SORE - Solder Reflow 
- moved on the sheet: C4, C6, J10, J4, J7, J8, R27, U3, U6A

Commit message: feat: routing part 2
Connections:
- net BCLK: now also J8.8 (Pin_8); no longer J8.7 (Pin_7)
- net CS0: now also J7.5 (Pin_5); no longer J10.10 (Pin_10)
- net DIO: now also J8.9 (Pin_9); no longer J8.10 (Pin_10)
- net I2C_SCL: now also J10.4 (Pin_4); no longer J10.7 (Pin_7)
- net I2C_SDA: now also J10.3 (Pin_3); no longer J10.6 (Pin_6)
- net IN1: now also J10.5 (Pin_5); no longer J7.5 (Pin_5)
- net IN2: now also J10.6 (Pin_6); no longer J7.6 (Pin_6)
- net IN3: now also J7.3 (Pin_3); no longer J8.8 (Pin_8)
- net IN4: now also J10.7 (Pin_7); no longer J7.9 (Pin_9)
- net IN5: now also J10.8 (Pin_8); no longer J7.10 (Pin_10)
- net IN6: now also J7.10 (Pin_10); no longer J8.1 (Pin_1)
- net IO5: now also J10.2 (Pin_2); no longer J10.5 (Pin_5)
- net IO8: now also J10.9 (Pin_9); no longer J10.8 (Pin_8)
- net MCLK: now also J8.7 (Pin_7); no longer J8.2 (Pin_2)
- net MISO: now also J7.8 (Pin_8); no longer J7.3 (Pin_3)
- net MOSI: now also J7.6 (Pin_6); no longer J7.1 (Pin_1)
- net MTCK: now also J8.6 (Pin_6); no longer J8.3 (Pin_3)
- net MTDI: now also J8.4 (Pin_4); no longer J8.5 (Pin_5)
- net MTDO: now also J8.5 (Pin_5); no longer J8.4 (Pin_4)
- net MTMS: now also J8.3 (Pin_3); no longer J8.6 (Pin_6)
- net PT100: now also J10.1 (Pin_1); no longer J10.4 (Pin_4)
- net QUADHD: now also J7.4 (Pin_4); no longer J10.9 (Pin_9)
- net QUADWP: now also J7.9 (Pin_9); no longer J7.4 (Pin_4)
- net RXD0: now also J8.2 (Pin_2); no longer J7.8 (Pin_8)
- net SCLK: now also J7.7 (Pin_7); no longer J7.2 (Pin_2)
- net SSRIN1: no longer J10.1 (Pin_1)
- net SSRIN2: no longer J10.2 (Pin_2)
- net TXD0: now also J8.1 (Pin_1); no longer J7.7 (Pin_7)
- net USB_D+: now also J7.1 (Pin_1)
- net USB_D-: now also J10.10 (Pin_10)
- net WS: now also J8.10 (Pin_10); no longer J8.9 (Pin_9)
- net ZC_INPUT: now also J7.2 (Pin_2); no longer J10.3 (Pin_3)

Commit message: feat: attempt to finish routing
Parts:
- removed J10: PINOUT, Connector_Molex:Molex_SL_171971-0010_1x10_P2.54mm_Vertical, symbol Connector_Generic:Conn_01x10
- removed J3: PTC_Con, TerminalBlock_Phoenix:TerminalBlock_Phoenix_PT-1,5-2-5.0-H_1x02_P5.00mm_Horizontal, symbol Connector:Screw_Terminal_01x02
- removed R12: 9K1, Resistor_SMD:R_0805_2012Metric_Pad1.20x1.40mm_HandSolder, symbol Device:R_US
- removed R13: 1K, Resistor_SMD:R_0805_2012Metric_Pad1.20x1.40mm_HandSolder, symbol Device:R_US
- removed R2, R4, R5, R6: 25k, Resistor_SMD:R_0805_2012Metric_Pad1.20x1.40mm_HandSolder, symbol Device:R_US
- removed R3: 2.5k, Resistor_SMD:R_0805_2012Metric_Pad1.20x1.40mm_HandSolder, symbol Device:R_US
- removed R8, R9: 16k, Resistor_SMD:R_0805_2012Metric_Pad1.20x1.40mm_HandSolder, symbol Device:R_US
- removed TH1: PT100, Package_TO_SOT_THT:TO-92-2_Horizontal2, symbol Sensor_Temperature:PT100
- removed U1: TL431LP, Package_TO_SOT_THT:TO-92_Inline_Wide, symbol Reference_Voltage:TL431LP
- removed U2: LM324, Package_SO:SOIC-14_3.9x8.7mm_P1.27mm, symbol Amplifier_Operational:LM324
- added C21: 100nF, Capacitor_SMD:C_0805_2012Metric_Pad1.18x1.45mm_HandSolder, symbol Device:C
- added J13: RTD_PT100, TerminalBlock_Phoenix:TerminalBlock_Phoenix_PT-1,5-3-5.0-H_1x03_P5.00mm_Horizontal, symbol Connector:Screw_Terminal_01x03
- added J3: PINOUT, Connector_Molex:Molex_SL_171971-0010_1x10_P2.54mm_Vertical, symbol Connector_Generic:Conn_01x10
- added JP2: 3_OR_2_Wire, Jumper:SolderJumper-3_P1.3mm_Open_RoundedPad1.0x1.5mm, symbol Jumper:SolderJumper_3_Open
- added JP3: 2_Wire, Jumper:SolderJumper-2_P1.3mm_Open_TrianglePad1.0x1.5mm, symbol Jumper:SolderJumper_2_Open
- added U9: MAX31865xTP, Package_DFN_QFN:TQFN-20-1EP_5x5mm_P0.65mm_EP3.25x3.25mm, symbol Sensor_Temperature:MAX31865xTP
- C1, C3: value 10nF -> 100nF
- R1: value 25k -> 400 1%
Connections:
- net +3.3V: now also C3.1, C21.1, U9.19 (DVDD), U9.20 (VDD)
- net +5V: no longer R1.2
- net CS0: now also J7.6 (Pin_6); no longer J7.5 (Pin_5)
- net GND: now also C21.2, JP2.3 (B), U9.10 (GND), U9.15 (DGND), U9.16 (GND), U9.21 (GND)
- net I2C_SCL: now also J3.4 (Pin_4)
- net I2C_SDA: now also J3.3 (Pin_3)
- net IN1: now also J3.5 (Pin_5)
- net IN2: now also J3.6 (Pin_6)
- net IN3: now also J7.8 (Pin_8); no longer J7.3 (Pin_3)
- net IN4: now also J3.7 (Pin_7)
- net IN5: now also J3.8 (Pin_8)
- net IN6: now also J7.1 (Pin_1); no longer J7.10 (Pin_10)
- net IO5: now also J3.2 (Pin_2), U9.18 (~{DRDY})
- net IO8: now also J3.9 (Pin_9), U9.13 (~{CS})
- net MISO: now also J7.3 (Pin_3), U9.14 (SDO); no longer J7.8 (Pin_8)
- net MOSI: now also J7.5 (Pin_5), U9.11 (SDI); no longer J7.6 (Pin_6)
- net PT100: now also J3.1 (Pin_1)
- net QUADHD: now also J7.7 (Pin_7); no longer J7.4 (Pin_4)
- net QUADWP: now also J7.2 (Pin_2); no longer J7.9 (Pin_9)
- net SCLK: now also J7.4 (Pin_4), U9.12 (SCLK); no longer J7.7 (Pin_7)
- net USB_D+: now also J7.10 (Pin_10); no longer J7.1 (Pin_1)
- net USB_D-: now also J3.10 (Pin_10)
- net ZC_INPUT: now also J7.9 (Pin_9); no longer J7.2 (Pin_2)
- net at C1.1: now also J13.2 (Pin_2), JP3.1 (A), U9.7 (RTDIN+)
- net at C1.2: now also J13.1 (Pin_1), U9.8 (RTDIN-), U9.9 (FORCE-)
- net +2V5: no longer names the net of R1.1
- net +2V5: now also U9.1 (BIAS), U9.2 (REFIN+)
- new net: R1.2, U9.3 (REFIN-), U9.4 (ISENSOR)
- new net: J13.3 (Pin_3), JP2.1 (A), JP3.2 (B), U9.5 (FORCE+)
- new net: JP2.2 (C), U9.6 (FORCE2)
Other:
- note added: "3 Wire to Force+ 2/4 Wire to GND Connect 2_Wire if use 2/4 Wire"
- note added: "Currently Excluded From Board"
- note removed: "Current Source 1mA"
- note removed: "Gain = 1 + (9,1K / 1K) = 10.1"
- note removed: "LM324 Vo=(1+R1/R2)*vref which: vref approx 2.5v R1=0 R2=~"
- note removed: "Output is limited by output range, which is typically 1.5 V to 10.5 V, or VCC- + 1.5 V to VCC+ - 1.5 V."
- note removed: "PT100-PREAMP"
- note removed: "Sallen-Key Filter http://sim.okawa-denshi.jp/en/OPstool.php"
- note removed: "Target Temp for PT100 is Less 400*C, Based on Resistance table its about 250ohm current source is 1mA, with tolerance, if resistance of PT100 300 ohm it will be 300mV, adding non inverting to increase gain into 3V (x10)"
- note removed: "if temp is not more than 400, voltage on pin 12 will never exeed 300mV"
- moved on the sheet: J7
