File: hardware/v2/solder-reflow.kicad_sch (KiCad schematic)
At the start: 111 parts, among them J1 USB_C_Receptacle_USB2.0_14P, J11 I2C, J12 JTAG10, J13 RTD_PT100, J14 SSROUT2, J15 LCD_CONN, J16 UART, J17 USB_C_Receptacle_USB2.0_14P, J18 High_To_Low_Link, J19 High_To_Low_Link, J2 I2S, J3 PINOUT, J4 220V, J5 HEATER, J6 InputButton, J7 PINOUT, J8 PINOUT, J9 12VIN, K1 G3MB202PDC12, Q1 SS8550, Q2 SS8550, Q3 SS8050, Q4 SS8050, SW1 L, SW2 RST, SW3 SWH11AA1, SW4 D, SW5 U, SW6 R, SW7 R, SW8 R, SW9 Boot, U3 L7805, U4 AMS1117-3.3, U5 ESP32-S3-WROOM-1, U6 74LS14, U7 H11AA1, U8 CH340C, U9 MAX31865xTP

Commit message: feat: change to use esp32-s3 tempel
Parts:
- removed C15: 22uF, Capacitor_SMD:C_0805_2012Metric_Pad1.18x1.45mm_HandSolder, symbol Device:C
- removed C16: 1uF, Capacitor_SMD:C_0805_2012Metric_Pad1.18x1.45mm_HandSolder, symbol Device:C
- removed C17, C18, C20: 100nF, Capacitor_SMD:C_0805_2012Metric_Pad1.18x1.45mm_HandSolder, symbol Device:C
- removed D3: TXD, LED_SMD:LED_1206_3216Metric_Pad1.42x1.75mm_HandSolder, symbol Device:LED
- removed D6: RXD, LED_SMD:LED_1206_3216Metric_Pad1.42x1.75mm_HandSolder, symbol Device:LED
- removed J1, J17: USB_C_Receptacle_USB2.0_14P, Connector_USB:USB_C_Receptacle_GCT_USB4110, symbol Connector:USB_C_Receptacle_USB2.0_14P
- removed J11: I2C, Connector_Molex:Molex_SL_171971-0004_1x04_P2.54mm_Vertical, symbol Connector_Generic:Conn_01x04
- removed J12: JTAG10, Connector_IDC:IDC-Header_2x05_P2.54mm_Vertical, symbol Connector:Conn_ARM_JTAG_SWD_10
- removed J16: UART, Connector_Molex:Molex_SL_171971-0004_1x04_P2.54mm_Vertical, symbol Connector_Generic:Conn_01x04
- removed J18, J19: High_To_Low_Link, Connector_IDC:IDC-Header_2x05_P2.54mm_Vertical, symbol Connector_Generic:Conn_02x05_Odd_Even
- removed J3, J7, J8: PINOUT, Connector_Molex:Molex_SL_171971-0010_1x10_P2.54mm_Vertical, symbol Connector_Generic:Conn_01x10
- removed Q3, Q4: SS8050, Package_TO_SOT_SMD:SOT-23_Handsoldering, symbol Transistor_BJT:BC817
- removed R10, R7: 4K7, Resistor_SMD:R_0805_2012Metric_Pad1.20x1.40mm_HandSolder, symbol Device:R_US
- removed R11, R21, R43, R44: 5K1, Resistor_SMD:R_0805_2012Metric_Pad1.20x1.40mm_HandSolder, symbol Device:R_US
- removed R22, R26, R28, R42: 1k, Resistor_SMD:R_0805_2012Metric_Pad1.20x1.40mm_HandSolder, symbol Device:R_US
- removed R45, R46: 10k, Resistor_SMD:R_0805_2012Metric_Pad1.20x1.40mm_HandSolder, symbol Device:R_US
- removed SW2: RST, Button_Switch_SMD:SW_Push_1P1T_NO_6x6mm_H9.5mm, symbol Switch:SW_Push
- removed SW9: Boot, Button_Switch_SMD:SW_Push_1P1T_NO_6x6mm_H9.5mm, symbol Switch:SW_Push
- removed U4: AMS1117-3.3, Package_TO_SOT_SMD:SOT-223-3_TabPin2, symbol Regulator_Linear:AMS1117-3.3
- removed U5: ESP32-S3-WROOM-1, RF_Module:ESP32-S3-WROOM-1U, symbol RF_Module:ESP32-S3-WROOM-1
- removed U8: CH340C, Package_SO:SOIC-16_3.9x9.9mm_P1.27mm, symbol Interface_USB:CH340C
- added J1: I2C, Connector_Molex:Molex_SL_171971-0004_1x04_P2.54mm_Vertical, symbol Connector_Generic:Conn_01x04
- added J3: RTD_PT100, TerminalBlock_Phoenix:TerminalBlock_Phoenix_PT-1,5-3-5.0-H_1x03_P5.00mm_Horizontal, symbol Connector:Screw_Terminal_01x03
- added JP4: 3_OR_2_Wire, Jumper:SolderJumper-3_P1.3mm_Open_RoundedPad1.0x1.5mm, symbol Jumper:SolderJumper_3_Open
- added JP5: 2_Wire, Jumper:SolderJumper-2_P1.3mm_Open_TrianglePad1.0x1.5mm, symbol Jumper:SolderJumper_2_Open
- added R2, R3: 4K7, Resistor_SMD:R_0805_2012Metric_Pad1.20x1.40mm_HandSolder, symbol Device:R_US
- added R4: 400 1%, Resistor_SMD:R_0805_2012Metric_Pad1.20x1.40mm_HandSolder, symbol Device:R_US
- added U1: ESP32-S3-Tempel, esp32-s3-tempel-lib:esp32-s3-tempel, symbol esp32-s3-tempel-lib:esp-32-s3-tempel
- added U2: MAX31865xTP, Package_DFN_QFN:TQFN-20-1EP_5x5mm_P0.65mm_EP3.25x3.25mm, symbol Sensor_Temperature:MAX31865xTP
- C11, C7: value 22uF -> 100nF
Connections:
- net +3.3V: now also C7.1, J1.1 (Pin_1), R2.2, R3.2, U1.35 (3V3), U2.19 (DVDD), U2.20 (VDD); no longer C14.1
- net +5V: now also U1.36 (5V); no longer C7.1
- net BCLK: now also U1.23 (IO45)
- net CS0: now also U1.15 (IO10)
- net DIO: now also U1.22 (IO48)
- net GND: now also J1.4 (Pin_4), JP4.3 (B), U1.34 (GND), U2.10 (GND), U2.15 (DGND), U2.16 (GND), U2.21 (GND); no longer C14.2
- net I2C_SCL: now also J1.3 (Pin_3), R3.1, U1.4 (IO7)
- net I2C_SDA: now also J1.2 (Pin_2), R2.1, U1.3 (IO6)
- net IN1: now also U1.5 (IO15)
- net IN2: now also U1.6 (IO16)
- net IN3: now also U1.13 (IO46)
- net IN4: now also U1.7 (IO17)
- net IN5: now also U1.8 (IO18)
- net IN6: now also U1.20 (IO21)
- net IO5: now also U9.13 (~{CS}), U1.2 (IO5), U2.18 (~{DRDY})
- net IO8: now also U1.9 (IO8); no longer U9.13 (~{CS})
- net MCLK: now also U1.25 (IO38)
- net MISO: now also U1.18 (IO13), U2.14 (SDO)
- net MOSI: now also U1.16 (IO11), U2.11 (SDI)
- net MTCK: now also U1.26 (IO39)
- net MTDI: now also U1.28 (IO41)
- net MTDO: now also U1.27 (IO40)
- net MTMS: now also U1.29 (IO42)
- net QUADHD: now also U1.14 (IO9)
- net QUADWP: now also U1.19 (IO14)
- net SCLK: now also U1.17 (IO12), U2.12 (SCLK)
- net SSRIN1: now also U1.33 (IO1)
- net SSRIN2: now also U1.32 (IO2)
- net WS: now also U1.21 (IO47)
- net ZC_INPUT: now also U1.12 (IO3)
- new net: C14.1, J3.2 (Pin_2), JP5.1 (A), U2.7 (RTDIN+)
- new net: C14.2, J3.1 (Pin_1), U2.8 (RTDIN-), U2.9 (FORCE-)
- new net: J3.3 (Pin_3), JP4.1 (A), JP5.2 (B), U2.5 (FORCE+)
- new net: JP4.2 (C), U2.6 (FORCE2)
- new net: R4.1, U2.1 (BIAS), U2.2 (REFIN+)
- new net: R4.2, U2.3 (REFIN-), U2.4 (ISENSOR)
- new net IO4: U1.1 (IO4), U2.13 (~{CS})
- no-connect marks 15 -> 7
Other:
- note added: "ESP32-S3 TEMPEL"
- note added: "This PinHeader Is Excluded from Board."
- note removed: "Currently Excluded From Board"
- note removed: "ESP32-S3"
- note removed: "High To Low Voltage Link"
- note removed: "JTAG"
- note removed: "PINOUT"
- note removed: "UART"
- note removed: "UART to USB"
- note removed: "USBC"
- moved on the sheet: C1, C10, C12, C13, C19, C2, C21, C3, C4, C5, C6, C8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

Commit message: feat: finish routing v3 prototype 1
Parts:
- added H3, H4: MountingHole_Pad, MountingHole:MountingHole_3.2mm_M3_DIN965_Pad, symbol Mechanical:MountingHole_Pad
- SW1, SW4, SW5, SW6, SW7, SW8: footprint Button_Switch_SMD:SW_Push_1P1T_NO_6x6mm_H9.5mm -> Button_Switch_SMD:SW_Push_1P1T_NO_CK_KMR2
Connections:
- net IO5: no longer U2.18 (~{DRDY}), U9.18 (~{DRDY})
- net MTDI renamed IO41
- net IO41: now also U2.18 (~{DRDY})
- net MTMS renamed IO42
- net IO42: now also U9.18 (~{DRDY})
- no-connect marks 7 -> 10
Other:
- note added: "Curently Excluded"

Commit message: feat: update schematic svg
Connections:
- no-connect marks 10 -> 9
