File: hardware/v3/sore_v3/sore_v3.kicad_sch (KiCad schematic)
At the start: 45 parts, among them J1 Barrel_Jack_Switch, Q1 WSP4409A, Q2 IRLR8726TRPBF, Q3 SS8050, U1 ATMEGA4809-AFR, U2 AMS1117-5.0

Commit message: copying pcb reflow schematic
Parts:
- added D5: WS2812B-2020, LED_SMD:LED_WS2812B-2020_PLCC4_2.0x2.0mm, symbol LED:WS2812B-2020
Other:
- moved on the sheet: C1, C11, C13, C2, C3, C4, C5, C6, C7, C8, C9, D1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
